File: Arachnode/hardware/Arachnode.brd (EAGLE design)
At the start: 71.1 x 33.7 mm, 39 parts, among them J1 PINHEAD-17-REV, J2 PINHEAD-17-REV, U1 BQ24210, U2 DS1337

Commit message: Modified ArachnNode to Arachnio Due standard
Parts:
- removed C3: 100n, resistor:C0603
- removed INTB, SQW: (no value), SparkFun-Passives:PAD-JUMPER-2-NO_YES_SILK
- removed R13, R14: 4k7, resistor:R0603
- removed U2: DS1337, SparkFun-FreqCtrl:SO08-TIGHT
- removed Y1: (no value), SparkFun-FreqCtrl:CRYSTAL-32KHZ-SMD_EPSON_MC146
Connections:
- removed net N$14: U2.2, Y1.P$1
- removed net N$15: INTB.2, R14.1, U2.3
- removed net N$2: R13.1, SQW.2, U2.7
- removed net N$4: U2.1, Y1.P$2
- net GND: no longer C3.2, U2.4
- net IO8: no longer SQW.1
- net IO9: no longer INTB.1
- net SCL: no longer U2.6
- net SDA: no longer U2.5
- net V_BATT: no longer C3.1, R13.2, R14.2, U2.8
Routing:
- net N$15: track 35.8 -> 0.00 mm, vias 2 -> 0
- net N$2: track 23.8 -> 0.00 mm, vias 2 -> 0
- net V_BATT: track 116.3 -> 105.1 mm, vias 8 -> 5
- net SCL: track 66.1 -> 57.4 mm, vias 3 -> 1
- net SDA: track 64.9 -> 59.4 mm, vias 3 -> 1
- net N$14: track 4.88 -> 0.00 mm
- net IO8: track 11.4 -> 7.80 mm
- net N$4: track 3.24 -> 0.00 mm
- net RESET: track 29.5 -> 26.7 mm
- net IO9: track 10.3 -> 8.25 mm
