File: ArachnoMoto/hardware/ArachnoMoto.brd (EAGLE design)
At the start: 74.9 x 60.3 mm, 32 parts, among them J1 PINHEAD-17-REV, J2 PINHEAD-17-REV, U1 DRV8801, U2 DRV8801, U3 USD-SOCKETNEW, X1 1751248, X2 1751248, X3 1751248, X4 1751248

Commit message: Ombnibus commit because I am not sure what I did...
Parts:
- added C10, C9: (no value), resistor:E5-10,5
- added LED1, LED2, LED3, LED4: (no value), adafruit:CHIP-LED0603
- added R4, R5, R8, R9: (no value), resistor:R0603
Connections:
- new net N$11: LED2.C, R5.1
- new net N$12: LED3.A, R8.1
- new net N$14: LED4.C, R9.1
- new net N$4: LED1.A, R4.1
- net GND: now also C10.-, C9.-
- net N$1: now also R8.2, R9.2
- net N$18: now also R4.2, R5.2
- net N$19: now also LED1.C, LED2.A
- net N$3: now also LED3.C, LED4.A
- net V+: now also C10.+, C9.+
Routing:
- net N$1: track 25.2 -> 45.8 mm, vias 0 -> 1
- net N$18: track 23.5 -> 41.4 mm, vias 0 -> 2
- net V+: track 190.9 -> 203.9 mm
- net N$19: track 30.3 -> 40.2 mm
- net N$3: track 29.6 -> 39.0 mm
- net N$12: track 0.00 -> 7.14 mm
- net N$11: track 0.00 -> 6.61 mm
- net N$4: track 0.00 -> 6.35 mm
- net N$14: track 0.00 -> 3.74 mm
- net MODE22: track 48.1 -> 47.2 mm
