File: ArachnioDue/hardware/ArachnioDue.brd (EAGLE design)
At the start: 17.8 x 58.4 mm, 62 parts, among them J5 HEAD17-NOSS, J6 HEAD17-NOSS, Q1 8MHz, T1 FDN340P/PMV48XP, U1 ATMEGA32U4-XUMU, U2 AP2111HA-3.3, U3 ZLDO1117-5.0, U5 ESP8266EX, U6 SPI_FLASH, Y1 26 MHz/10 pF

Commit message: -- Captured schematic for SAM3S*A version
Parts:
- removed C15: 10u/6.3V, resistor:C0603
- removed GPIO0, GPIO2, MTDO, OTA: JUMPER-PAD-2-NOYES_SILK, SparkFun-Passives:PAD-JUMPER-2-NO_YES_SILK
- removed L2: MH2029-300Y, wuerth-elektronik:0805
- removed R12: 0R, resistor:R0603
- removed R4: 10K, resistor:R0603
- removed R6: 1K, resistor:R0603
- removed T1: FDN340P/PMV48XP, zetex:SOT-23
- removed TX: YLW, led:CHIP-LED0603
- removed U3: ZLDO1117-5.0, logos-power:SOT223
- added C12, C13, C2, C20, C21, C22, C27, C28, C29: 100n, resistor:C0402
- added C14: 2u2, resistor:C0603
- added C23, C24, C25, C26: 4u7, resistor:C0603
- added D1, D2: CGRM4001-G, diode:SOD-123_MINI-SMA
- added ERASE: (no value), adafruit:KMR2
- added L1: 10u/100mA, wuerth-elektronik:0805
- added LOAD/OTA: (no value), SparkFun-Passives:PAD-JUMPER-3-NO_YES_SILK
- added RST: (no value), SparkFun-Passives:PAD-JUMPER-2-NC_BY_TRACE_YES_SILK
- added Y2: (no value), SparkFun-FreqCtrl:CRYSTAL-32KHZ-SMD_EPSON_MC146
- C10, C6: value 100n -> 4u7
- C11, C16, C17, C18, C19: device resistor:C0603 -> resistor:C0402
- C5: value 1uF -> 100n; device resistor:C0603 -> resistor:C0402
- C7: value 1uF -> 4u7
- CN1: device adafruit:USB-MINIB -> SparkFun-Connectors:USB-AB-MICRO-SMD
- Q1: value 8MHz -> 12MHz
- R1, R10, R11, R13, R14, R2, R3, R5, R7, R8, R9: device resistor:R0603 -> resistor:R0402
- RESET: value SPST_TACT-KMR2 -> (none)
- RN1: value 22R -> 27R
- U1: value ATMEGA32U4-XUMU -> SAM3SA-MU; device SmartPrj:QFN44ML7X7 -> atmel-sam3s:QFN48
- moved TP2 224.4 mm to (-49.8, -166.6), flipped to the top, turned to 0 degrees
- moved TP1 220.0 mm to (-49.8, -162.6), flipped to the top, turned to 0 degrees
- moved R9 205.6 mm to (-49.5, -157.5), flipped to the top, turned to 0 degrees
- moved C7 117.9 mm to (-45.7, -76.2), flipped to the top, turned to 0 degrees
- moved C10 113.4 mm to (-45.7, -81.3), turned to 0 degrees
- moved C5 107.7 mm to (-45.7, -61.6)
- moved C6 106.0 mm to (-45.7, -66.7), turned to 0 degrees
- moved U2 25.5 mm to (35.4, 21.0)
- moved C1 24.3 mm to (29.8, 21.0)
- moved C19 23.5 mm to (31.8, 38.1)
- moved RX 23.0 mm to (36.2, 29.3)
- moved U6 21.0 mm to (-13.8, 40.0)
- moved R5 19.1 mm to (-7.62, 6.99)
- moved L 19.1 mm to (32.4, 16.3)
- moved R14 18.5 mm to (-13.3, 45.5)
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Connections:
- removed net +5V: C3.1, J6.6, R5.1, T1.2, U2.3, U3.2, U3.4
- removed net AVCC: C7.1, L2.2, U1.44
- removed net CHIP_EN: J6.7, R11.2, U5.7
- removed net D4*: J5.9, U1.25
- removed net D5*: J5.10, U1.31
- removed net D6*: J5.11, U1.27
- removed net D7: J5.12, U1.1
- removed net ESP_RST: J6.8, R12.2, R14.2, U5.8
- removed net HWB: R4.1, U1.33
- removed net IO10*: J5.15, U1.30
- removed net IO11*: J5.16, U1.12
- removed net IO12*: J5.17, U1.26
- removed net IO13: J6.17, R8.1, U1.32
- removed net IO8: J5.13, U1.28
- removed net IO9*: J5.14, U1.29
- removed net N$4: R6.2, TX.A
- removed net RXLED/SS: J5.2, R7.1, U1.8
- removed net TXLED: R6.1, U1.22
- removed net UCAP: C5.1, U1.6
- new net D10: J5.15, U1.15
- new net D11: J5.16, U1.35
- new net D12: J5.17, U1.32
- new net D13: J6.17, R8.1, U1.36
- new net D4: J5.9, U1.5
- new net D5: J5.10, U1.25
- new net D6: J5.11, U1.6
- new net D8: J5.13
- new net D9: J5.14, U1.20
- new net ERASE: ERASE.2, ERASE.4, J6.7, R9.2, U1.42
- new net ESP_RX: TP2.TP, U1.21, U5.25
- new net ESP_TX: TP1.TP, U1.22, U5.26
- new net N$8: C3.1, C4.1, D1.C, D2.C, U2.3
- new net RXTXLED/SS: J5.2, R7.1, U1.14
- new net SWCLK/D8: U1.40
- new net SWDIO/D7/CHIP_EN: J5.12, R11.2, U1.39, U5.7
- new net SWO/ESP_RST: J6.8, R14.2, RST.2, U1.37, U5.8
- new net VDDOUT: C13.1, C14.1, L1.1, U1.18, U1.41, U1.8
- new net VDDPLL: C2.1, C5.1, C6.1, L1.2, U1.48
- net 3V3: now also C20.1, C21.1, C22.1, C23.1, C24.1, C25.1, C26.1, C27.1, C28.1, C29.1, C7.1, ERASE.1, ERASE.3, R10.2, R5.1, RX.A, U1.13, U1.33, U1.47, U1.7, U5.14; no longer C15.1, L2.1, U1.14, U1.2, U1.24, U1.34
- net A0: now also U1.9; no longer U1.36
- net A1: now also U1.10; no longer U1.37
- net A2: now also U1.11; no longer U1.38
- net A3: now also U1.12; no longer U1.39
- net A4: now also U1.3; no longer U1.40
- net A5: now also U1.4; no longer U1.41
- net AREF: now also C12.2, U1.1; no longer C6.1, U1.42
- net D0/RX: now also U1.27; no longer U1.20, U5.26
- net D1/TX: now also U1.26; no longer U1.21, U5.25
- net D2/SDA: now also U1.31; no longer GPIO2.2, U1.19
- net D3/SCL: now also LOAD/OTA.3, U1.28; no longer GPIO0.2, U1.18
- net GND: now also C12.1, C13.2, C14.2, C2.2, C20.2, C21.2, C22.2, C23.2, C24.2, C25.2, C26.2, C27.2, C28.2, C29.2, U1.2, U1.30, U1.34, U5.13; no longer C15.2, R10.1, R4.2, RX.C, TX.C, U1.15, U1.23, U1.35, U1.43, U1.5, U1.EXP, U3.1
- net MISO: now also U1.19; no longer U1.11
- net MOSI: now also U1.17; no longer MTDO.2, U1.10
- net N$1: now also U1.23, Y2.P$2; no longer MTDO.1, R10.2, TP1.TP, U5.13
- net N$2: now also RX.C; no longer RX.A
- net N$33: now also RST.1; no longer R12.1
- net N$5: now also U1.24, Y2.P$1; no longer GPIO2.1, TP2.TP, U5.14
- net N$6: now also LOAD/OTA.2, R10.1; no longer GPIO0.1, OTA.1
- net RD+: now also U1.44; no longer U1.4
- net RD-: now also U1.43; no longer U1.3
- net RESET: now also LOAD/OTA.1, U1.29; no longer OTA.2, U1.13
- net SCK: now also U1.16; no longer U1.9
- net VIN: now also D2.A; no longer C4.1, R9.2, T1.3, U3.3
- net VUSB: now also D1.A, J6.6; no longer T1.1, U1.7
- net XTAL1: now also U1.46; no longer U1.17
- net XTAL2: now also U1.45; no longer U1.16
Routing:
- net 3V3: track 66.9 -> 0.00 mm, vias 12 -> 0
- net +5V: track 43.2 -> 0.00 mm, vias 2 -> 0
- net VIN: track 41.1 -> 0.00 mm, vias 1 -> 0
- net VUSB: track 38.4 -> 0.00 mm, vias 1 -> 0
- net RESET: track 35.3 -> 0.00 mm, vias 1 -> 0
- net D1/TX: track 32.9 -> 0.00 mm, vias 3 -> 0
- net D0/RX: track 31.6 -> 0.00 mm, vias 3 -> 0
- net ESP_RST: track 30.6 -> 0.00 mm, vias 2 -> 0
- net D7: track 30.0 -> 0.00 mm, vias 2 -> 0
- net IO11*: track 30.0 -> 0.00 mm, vias 1 -> 0
- net GND: track 27.0 -> 0.00 mm, vias 38 -> 0
- net CHIP_EN: track 25.9 -> 0.00 mm, vias 2 -> 0
- net IO13: track 24.5 -> 0.00 mm
- net MOSI: track 23.3 -> 0.00 mm, vias 1 -> 0
- net IO12*: track 23.1 -> 0.00 mm, vias 1 -> 0
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
Commit message: ﻿First test boards of this design # Please enter the commit message for your changes. Lines starting # with '#' will be ignored, and an empty message aborts the commit. # On branch master # Your branch is ahead of 'origin/master' by 1 commit. #   (use "git push" to publish your local commits) # # Changes to be committed: #	new file:   ArachnioDue/hardware/ArachnioDue.G15L #	new file:   ArachnioDue/hardware/ArachnioDue.G2L #	new file:   ArachnioDue/hardware/ArachnioDue.GBL #	new file:   ArachnioDue/hardware/ArachnioDue.GBO #	new file:   ArachnioDue/hardware/ArachnioDue.GBS #	new file:   ArachnioDue/hardware/ArachnioDue.GDM #	new file:   ArachnioDue/hardware/ArachnioDue.GML #	new file:   ArachnioDue/hardware/ArachnioDue.GTL #	new file:   ArachnioDue/hardware/ArachnioDue.GTO #	new file:   ArachnioDue/hardware/ArachnioDue.GTS #	new file:   ArachnioDue/hardware/ArachnioDue.TXT #	modified:   ArachnioDue/hardware/ArachnioDue.brd #	new file:   ArachnioDue/hardware/ArachnioDue.gcb #	new file:   ArachnioDue/hardware/ArachnioDue.gct #	new file:   ArachnioDue/hardware/ArachnioDue.oln #	modified:   ArachnioDue/hardware/ArachnioDue.sch #	new file:   ArachnioDue/hardware/ArachnioDue.zip #
Parts:
- removed TP1, TP2: PTR1TP15SQ, testpad:TP15SQ
- added C15: 100n, resistor:C0402
- D1, D2: value CGRM4001-G -> (none); device diode:SOD-123_MINI-SMA -> SparkFun-DiscreteSemi:SOD-123
- moved R9 201.5 mm to (5.59, 36.3)
- moved LOAD/OTA 200.5 mm to (4.83, 40.6)
- moved C24 157.9 mm to (7.11, 21.8), flipped to the bottom, turned to 180 degrees
- moved C23 154.6 mm to (7.11, 23.4), flipped to the bottom, turned to 180 degrees
- moved C21 151.9 mm to (11.7, 28.8), turned to 90 degrees
- moved C22 146.2 mm to (3.56, 20.8), turned to 270 degrees
- moved C14 137.1 mm to (10.7, 23.4), flipped to the bottom
- moved C13 136.8 mm to (9.14, 28.8), turned to 90 degrees
- moved C20 135.9 mm to (11.2, 16.8), turned to 270 degrees
- moved C12 126.2 mm to (14.2, 19.6), turned to 270 degrees
- moved C10 116.2 mm to (10.7, 20.3), flipped to the bottom
- moved C7 113.1 mm to (10.7, 21.8), flipped to the bottom
- moved L1 106.4 mm to (14.2, 17.3), flipped to the bottom, turned to 90 degrees
- moved C6 102.3 mm to (12.7, 17.3), flipped to the bottom, turned to 270 degrees
- moved C5 98.7 mm to (14.2, 16.8), turned to 270 degrees
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Connections:
- removed net D8: J5.13
- removed net ESP_RX: TP2.TP, U1.21, U5.25
- removed net ESP_TX: TP1.TP, U1.22, U5.26
- removed net N$8: C3.1, C4.1, D1.C, D2.C, U2.3
- removed net SWDIO/D7/CHIP_EN: J5.12, R11.2, U1.39, U5.7
- new net CHIP_EN: R11.2, U1.15, U5.7
- new net SWDIO/D7: J5.12, U1.39
- new net VCC: C3.1, C4.1, D1.C, D2.C, J6.6, U2.3
- net D0/RX: now also U1.22, U5.26; no longer U1.27
- net D1/TX: now also U1.21, U5.25; no longer U1.26
- net D10: now also U1.32; no longer U1.15
- net D12: now also U1.20; no longer U1.32
- net D4: now also U1.6; no longer U1.5
- net D6: now also U1.5; no longer U1.6
- net D9: now also U1.27; no longer U1.20
- net GND: now also C15.2
- net SWCLK/D8: now also J5.13
- net VDDOUT: now also C15.1
- net VUSB: no longer J6.6
Routing:
- net 3V3: track 0.00 -> 58.6 mm, vias 0 -> 17
- net SWO/ESP_RST: track 0.00 -> 52.4 mm, vias 0 -> 2
- net RESET: track 0.00 -> 38.7 mm, vias 0 -> 2
- net ERASE: track 0.00 -> 37.1 mm, vias 0 -> 4
- net VCC: track 0.00 -> 35.9 mm
- net D0/RX: track 0.00 -> 32.9 mm, vias 0 -> 2
- net D1/TX: track 0.00 -> 32.4 mm, vias 0 -> 2
- net VDDOUT: track 0.00 -> 30.6 mm, vias 0 -> 4
- net D12: track 0.00 -> 27.9 mm, vias 0 -> 1
- net CHIP_EN: track 0.00 -> 26.5 mm, vias 0 -> 2
- net MOSI: track 0.00 -> 25.1 mm, vias 0 -> 1
- net RXTXLED/SS: track 0.00 -> 23.7 mm, vias 0 -> 4
- net D13: track 0.00 -> 22.6 mm
- net SCK: track 0.00 -> 21.4 mm, vias 0 -> 1
- net D3/SCL: track 0.00 -> 21.0 mm, vias 0 -> 1
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Other:
- board text added: "ERASE"
- board text added: "V+"
- board text removed: "5V"
- board text removed: "EN"
- board text removed: "L"
- board text removed: "PWR"

Commit message: first module version, ready for mfg
Parts:
- removed C16, C17: 10 pF, resistor:C0402
- removed C18: 5p6, resistor:C0402
- removed C19, C27, C28, C29: 100n, resistor:C0402
- removed C25, C26: 4u7, resistor:C0603
- removed LOAD/OTA: (no value), SparkFun-Passives:PAD-JUMPER-3-NO_YES_SILK
- removed R10, R11, R14: 10K, resistor:R0402
- removed R13: 200R, resistor:R0402
- removed R3: 12K, resistor:R0402
- removed RST: (no value), SparkFun-Passives:PAD-JUMPER-2-NC_BY_TRACE_YES_SILK
- removed TP3: PTR1TP15SQ, testpad:TP15SQ
- removed U$11: ANTENNA_1RIGHT, ant-planar-1:SWRA117D_RIGHT
- removed U5: ESP8266EX, ESP8266:QFN32
- removed U6: SPI_FLASH, ESP8266:SOIC-8
- removed Y1: 26 MHz/10 pF, SmartPrj:CRYSTAL-3.2-2.5
- added ERASE_JMP, RST_JMP: JUMPER-PAD-2-NOYES_SILK, SparkFun-Passives:PAD-JUMPER-2-NO_YES_SILK
- added ESP1: ESP-12, esp8266-parts:ESP-12
- J5: value HEAD17-NOSS -> (none); device SmartPrj:HEAD17-NOSS -> logos-headers:1X17SMD-UNIVERSAL
- J6: device SmartPrj:HEAD17-NOSS-1 -> logos-headers:1X17SMD-UNIVERSAL
- U1: value SAM3SA-MU -> SAM3SB-AU; device atmel-sam3s:QFN48 -> atmel-sam3s:LQFP64
- moved R9 21.8 mm to (7.62, 14.6), turned to 90 degrees
- moved ERASE 19.8 mm to (1.91, 14.6), turned to 90 degrees
- moved U$12 15.1 mm to (17.1, 48.3)
- moved U$37 12.3 mm to (16.5, 2.29)
- moved C15 10.2 mm to (17.1, 12.1), turned to 180 degrees
- moved RX 9.26 mm to (-0.64, 37.5), turned to 0 degrees
- moved C13 9.03 mm to (17.1, 24.6), turned to 0 degrees
- moved U$1 6.25 mm to (14.6, 41.3)
- moved R7 5.26 mm to (-0.64, 40.0), turned to 270 degrees
- moved RESET 4.70 mm to (15.9, 31.1), turned to 270 degrees
- moved C6 4.66 mm to (17.1, 15.9), flipped to the top, turned to 0 degrees
- moved C2 4.46 mm to (17.1, 17.1), turned to 0 degrees
- moved L1 4.41 mm to (17.1, 14.0), flipped to the top, turned to 180 degrees
- moved C8 4.15 mm to (12.1, 6.35), turned to 90 degrees
- moved C1 3.97 mm to (10.2, 19.7)
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Connections:
- removed net DVDD: U5.24
- removed net N$27: C17.1, U5.28, Y1.1
- removed net N$28: C16.1, U5.27, Y1.3
- removed net N$31: C18.1, U$11.RF
- removed net N$32: R3.1, U5.31
- removed net N$33: RST.1, U5.32
- removed net N$34: R13.2, U5.21
- removed net N$35: R13.1, U6.6
- removed net N$36: U5.20, U6.1
- removed net N$37: U5.18, U6.7
- removed net N$38: U5.19, U6.3
- removed net N$39: U5.23, U6.5
- removed net N$40: U5.22, U6.2
- removed net N$45: C18.2, U5.2
- removed net N$6: LOAD/OTA.2, R10.1, TP3.TP, U5.15
- removed net SWO/ESP_RST: J6.8, R14.2, RST.2, U1.37, U5.8
- removed net VDD: U5.16
- removed net VDD_RTC: U5.5
- new net ESP_CS: ESP1.CS, U1.15
- new net ESP_INT: ESP1.INT, U1.23
- new net ESP_LOAD: ESP1.GPIO0
- new net ESP_RESET: ESP1.REST
- new net ESP_RX: ESP1.TXD, U1.11
- new net ESP_TX: ESP1.RXD, U1.14
- new net N$4: ESP1.GPIO13, RST_JMP.2
- new net N$8: ERASE_JMP.1, ESP1.GPIO12
- new net SWO: J6.8, U1.49
- net 3V3: now also ESP1.VCC, U1.18, U1.45, U1.58; no longer C19.1, C25.1, C26.1, C27.1, C28.1, C29.1, R10.2, R11.1, R14.1, U1.13, U1.33, U1.47, U5.1, U5.11, U5.14, U5.17, U5.29, U5.3, U5.30, U5.4, U6.8
- net A2: now also U1.13; no longer U1.11
- net A3: now also U1.16; no longer U1.12
- net CHIP_EN: now also U1.20; no longer R11.2, U1.15, U5.7
- net D0/RX: now also U1.30; no longer U1.22, U5.26
- net D1/TX: now also U1.29; no longer U1.21, U5.25
- net D10: now also U1.44; no longer U1.32
- net D11: now also U1.47; no longer U1.35
- net D12: now also U1.28; no longer U1.20
- net D13: now also U1.48; no longer U1.36
- net D2/SDA: now also U1.43; no longer U1.31
- net D3/SCL: now also U1.36; no longer LOAD/OTA.3, U1.28
- net D5: now also U1.33; no longer U1.25
- net D9: now also U1.35; no longer U1.27
- net ERASE: now also ERASE_JMP.2, U1.55; no longer U1.42
- net GND: now also ESP1.GND, U1.17, U1.40, U1.46, U1.60; no longer C16.2, C17.2, C19.2, C25.2, C26.2, C27.2, C28.2, C29.2, R3.2, U$11.GND, U1.30, U1.34, U5.13, U5.33, U6.4, Y1.2, Y1.4
- net MISO: now also ESP1.MOSI, U1.27; no longer U1.19
- net MOSI: now also ESP1.MISO, U1.22; no longer U1.17
- net N$1: now also U1.31; no longer U1.23
- net N$5: now also U1.32; no longer U1.24
- net RD+: now also U1.57; no longer U1.44
- net RD-: now also U1.56; no longer U1.43
- net RESET: now also RST_JMP.1, U1.39; no longer LOAD/OTA.1, U1.29
- net RXTXLED/SS: now also U1.19; no longer U1.14
- net SCK: now also ESP1.CLK, U1.21; no longer U1.16
- net SWCLK/D8: now also U1.53; no longer U1.40
- net SWDIO/D7: now also U1.51; no longer U1.39
- net VDDOUT: now also U1.12, U1.24; no longer U1.18, U1.41
- net VDDPLL: now also U1.64; no longer U1.48
- net XTAL1: now also U1.62; no longer U1.46
- net XTAL2: now also U1.61; no longer U1.45
Routing:
- net SWO/ESP_RST: track 52.4 -> 0.00 mm, vias 2 -> 0
- net ESP_RX: track 0.00 -> 34.5 mm, vias 0 -> 2
- net ERASE: track 37.1 -> 69.8 mm, vias 4 -> 3
- net ESP_TX: track 0.00 -> 28.6 mm, vias 0 -> 2
- net CHIP_EN: track 26.5 -> 0.00 mm, vias 2 -> 0
- net SWO: track 0.00 -> 20.8 mm, vias 0 -> 3
- net 3V3: track 58.6 -> 40.1 mm, vias 17 -> 10
- net D0/RX: track 32.9 -> 14.7 mm, vias 2 -> 1
- net D3/SCL: track 21.0 -> 3.31 mm
- net ESP_CS: track 0.00 -> 16.8 mm, vias 0 -> 2
- net D1/TX: track 32.4 -> 16.3 mm, vias 2 -> 3
- net N$6: track 15.0 -> 0.00 mm, vias 1 -> 0
- net SCK: track 21.4 -> 36.1 mm, vias 1 -> 3
- net N$27: track 11.6 -> 0.00 mm
- net VCC: track 35.9 -> 47.5 mm, vias 0 -> 2
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Other:
- board size 17.8 x 58.4 mm -> 21.6 x 52.1 mm
- board text removed: "ERASE"
- board text removed: "RX"
